Commit message: Update workspace.

File: src/balance_description/urdf/balance.urdf.xacro (robot description, xacro)
@@ -2,8 +2,8 @@
 <robot xmlns:xacro="http://www.ros.org/wiki/xacro" name="diffbot">
     <!-- Constants for robot dimensions -->
-    <xacro:property name="mass" value="10.0"/> <!-- 增加质量 -->
+    <xacro:property name="mass" value="2.0"/> <!-- 增加质量 -->
     <xacro:property name="width" value="0.5"/> <!-- Square dimensions (widthxwidth) of beams -->
     <xacro:property name="length" value="0.5"/>
-    <xacro:property name="height" value="0.08"/>
+    <xacro:property name="height" value="0.061"/>
     <xacro:property name="wheel_length" value="0.03"/> <!-- Link 1 -->
     <xacro:property name="wheel_radius" value="0.1"/> <!-- Link 2 -->
@@ -39,7 +39,8 @@
       </visual>
       <inertial>
+        <!--质心位置在此修改 0.001 0.0 0.0-->
         <origin xyz="0.0 0.0 0.0" rpy="0.0 0.0 0.0"/>
         <mass value="${mass}"/>
-        <inertia ixx="0.21367" ixy="0.0" ixz="0.0" iyy="0.21367" iyz="0.0" izz="0.41667"/>
+        <inertia ixx="0.04229" ixy="0.0" ixz="0.0" iyy="0.04229" iyz="0.0" izz="0.08333"/>
       </inertial>
       <collision>
@@ -50,4 +51,22 @@
       </collision>
     </link>
+    <!-- IMU Link -->
+    <link name="imu_link">
+      <visual>
+        <geometry>
+          <box size="0.01 0.01 0.01"/>
+        </geometry>
+      </visual>
+      <inertial>
+        <mass value="0.001"/>
+        <origin xyz="0 0 0" rpy="0 0 0"/>
+        <inertia ixx="0.000001" ixy="0" ixz="0" iyy="0.000001" iyz="0" izz="0.000001"/>
+      </inertial>
+    </link>
+    <joint name="imu_joint" type="fixed">
+      <parent link="base_link"/>
+      <child link="imu_link"/>
+      <origin xyz="0 0 0" rpy="0 0 0"/>
+    </joint>
     <xacro:macro name="wheel" params="prefix reflect num">
       <link name="${prefix}_wheel">
@@ -70,11 +89,11 @@
       </link>
       <joint name="${prefix}_wheel_joint" type="continuous">
-        <origin xyz="0.0 ${reflect*(width/2+wheel_length/2)} 0.0" rpy="${-pi/2} 0.0 0.0"/>
+        <origin xyz="0.0 ${reflect*(width/2+wheel_length/2)} ${-height/3}" rpy="${-pi/2} 0.0 0.0"/>
         <parent link="base_link"/>
         <child link="${prefix}_wheel"/>
         <axis xyz="0.0 0.0 1"/>
-        <limit effort="3.07" velocity="73.7"/>
+        <limit effort="103.07" velocity="173.7" upper_limit="1e10" lower_limit="-1e10"/>
         <!-- 添加动力学属性：damping 为粘性阻尼，friction 为静摩擦力 -->
-        <dynamics damping="0.1" friction="0.1"/>
+        <dynamics damping="0.01" friction="0.01"/>
       </joint>
       <transmission name="${prefix}_wheel_trans">
@@ -90,4 +109,23 @@
     <xacro:wheel prefix="left" num="0" reflect="1"/>
     <xacro:wheel prefix="right" num="1" reflect="-1"/>
+    <gazebo reference="imu_link">
+      <gravity>true</gravity>
+      <sensor name="imu_sensor" type="imu">
+        <always_on>true</always_on>
+        <update_rate>100</update_rate>
+        <visualize>true</visualize>
+        <imu/>
+        <plugin filename="libgazebo_ros_imu_sensor.so" name="imu_plugin">
+          <topicName>imu</topicName>
+          <bodyName>imu_link</bodyName>
+          <updateRateHZ>100.0</updateRateHZ>
+          <gaussianNoise>0.0</gaussianNoise>
+          <xyzOffset>0 0 0</xyzOffset>
+          <rpyOffset>0 0 0</rpyOffset>
+          <frameName>imu_link</frameName>
+          <initialOrientationAsReference>false</initialOrientationAsReference>
+        </plugin>
+      </sensor>
+    </gazebo>
     <gazebo>
       <plugin name="gazebo_ros_control" filename="libgazebo_ros_control.so">

Commit message: Modified the balancing car URDF.

File: src/balance_description/urdf/balance.urdf.xacro (robot description, xacro)
@@ -89,5 +89,5 @@
       </link>
       <joint name="${prefix}_wheel_joint" type="continuous">
-        <origin xyz="0.0 ${reflect*(width/2+wheel_length/2)} ${-height/3}" rpy="${-pi/2} 0.0 0.0"/>
+        <origin xyz="0.0 ${reflect*(width/2+wheel_length/2)} ${-height*2}" rpy="${-pi/2} 0.0 0.0"/>
         <parent link="base_link"/>
         <child link="${prefix}_wheel"/>

Commit message: Update avalible lqr controller.

File: src/balance_description/urdf/balance.urdf.xacro (robot description, xacro)
@@ -89,9 +89,9 @@
       </link>
       <joint name="${prefix}_wheel_joint" type="continuous">
-        <origin xyz="0.0 ${reflect*(width/2+wheel_length/2)} ${-height*2}" rpy="${-pi/2} 0.0 0.0"/>
+        <origin xyz="0.0 ${reflect*(width/2+wheel_length/2)} ${-height*5}" rpy="${-pi/2} 0.0 0.0"/>
         <parent link="base_link"/>
         <child link="${prefix}_wheel"/>
         <axis xyz="0.0 0.0 1"/>
-        <limit effort="103.07" velocity="173.7" upper_limit="1e10" lower_limit="-1e10"/>
+        <limit effort="3.07" velocity="73.7" upper_limit="1e10" lower_limit="-1e10"/>
         <!-- 添加动力学属性：damping 为粘性阻尼，friction 为静摩擦力 -->
         <dynamics damping="0.01" friction="0.01"/>
@@ -113,5 +113,5 @@
       <sensor name="imu_sensor" type="imu">
         <always_on>true</always_on>
-        <update_rate>100</update_rate>
+        <update_rate>1000</update_rate>
         <visualize>true</visualize>
         <imu/>

Commit message: Update a pair of beautiful config yaml

File: src/balance_description/urdf/balance.urdf.xacro (robot description, xacro)
@@ -89,9 +89,9 @@
       </link>
       <joint name="${prefix}_wheel_joint" type="continuous">
-        <origin xyz="0.0 ${reflect*(width/2+wheel_length/2)} ${-height*2}" rpy="${-pi/2} 0.0 0.0"/>
+        <origin xyz="0.0 ${reflect*(width/2+wheel_length/2)} ${-height*5}" rpy="${-pi/2} 0.0 0.0"/>
         <parent link="base_link"/>
         <child link="${prefix}_wheel"/>
         <axis xyz="0.0 0.0 1"/>
-        <limit effort="103.07" velocity="173.7" upper_limit="1e10" lower_limit="-1e10"/>
+        <limit effort="3.07" velocity="73.7" upper_limit="1e10" lower_limit="-1e10"/>
         <!-- 添加动力学属性：damping 为粘性阻尼，friction 为静摩擦力 -->
         <dynamics damping="0.01" friction="0.01"/>

Commit message: Add a gimbal with yaw and pitch for balance car

File: src/balance_description/urdf/balance.urdf.xacro (robot description, xacro)
@@ -8,8 +8,8 @@
     <xacro:property name="wheel_length" value="0.03"/> <!-- Link 1 -->
     <xacro:property name="wheel_radius" value="0.1"/> <!-- Link 2 -->
-    <xacro:property name="gimbal_height" value="0.03"/>
-    <xacro:property name="gimbal_radius" value="0.02"/>
-    <xacro:property name="muzzle_height" value="0.05"/>
-    <xacro:property name="muzzle_radius" value="0.01"/>
+    <xacro:property name="gimbal_height" value="0.12"/>
+    <xacro:property name="gimbal_radius" value="0.06"/>
+    <xacro:property name="muzzle_height" value="0.4"/>
+    <xacro:property name="muzzle_radius" value="0.03"/>
     <material name="orange">
       <color rgba="${255/255} ${108/255} ${10/255} 1.0"/>
@@ -39,6 +39,6 @@
       </visual>
       <inertial>
-        <!--质心位置在此修改 0.001 0.0 0.0-->
-        <origin xyz="0.0 0.0 0.0" rpy="0.0 0.0 0.0"/>
+        <!-- 质心偏移计算结果为 -0.015 以配平 muzzle 的 0.03 偏移 -->
+        <origin xyz="-0.015 0.0 0.0" rpy="0.0 0.0 0.0"/>
         <mass value="${mass}"/>
         <inertia ixx="0.04229" ixy="0.0" ixz="0.0" iyy="0.04229" iyz="0.0" izz="0.08333"/>
@@ -67,4 +67,21 @@
       <parent link="base_link"/>
       <child link="imu_link"/>
+      <origin xyz="0 0 0" rpy="0 0 0"/>
+    </joint>
+    <link name="gimbal_imu_link">
+      <visual>
+        <geometry>
+          <box size="0.01 0.01 0.01"/>
+        </geometry>
+      </visual>
+      <inertial>
+        <mass value="0.001"/>
+        <origin xyz="0 0 0" rpy="0 0 0"/>
+        <inertia ixx="0.000001" ixy="0" ixz="0" iyy="0.000001" iyz="0" izz="0.000001"/>
+      </inertial>
+    </link>
+    <joint name="gimbal_imu_joint" type="fixed">
+      <parent link="muzzle_link"/>
+      <child link="gimbal_imu_link"/>
       <origin xyz="0 0 0" rpy="0 0 0"/>
     </joint>
@@ -103,4 +120,5 @@
         </joint>
         <actuator name="${prefix}_wheel_motor">
+          <hardwareInterface>hardware_interface/EffortJointInterface</hardwareInterface>
           <mechanicalReduction>1</mechanicalReduction>
         </actuator>
@@ -109,4 +127,98 @@
     <xacro:wheel prefix="left" num="0" reflect="1"/>
     <xacro:wheel prefix="right" num="1" reflect="-1"/>
+    <link name="gimbal_link">
+      <inertial>
+        <origin xyz="0.0 0.0 0.0" rpy="0.0 0.0 0.0"/>
+        <mass value="0.2"/>
+        <inertia ixx="0.00042" ixy="0.0" ixz="0.0" iyy="0.00042" iyz="0.0" izz="0.00036"/>
+      </inertial>
+      <visual name="">
+        <origin xyz="0.0 0.0 0.0" rpy="0.0 0.0 0.0"/>
+        <geometry>
+          <cylinder radius="${gimbal_radius}" length="${gimbal_height}"/>
+        </geometry>
+        <material name="white"/>
+      </visual>
+      <collision>
+        <origin xyz="0.0 0.0 0.0" rpy="0.0 0.0 0.0"/>
+        <geometry>
+          <cylinder radius="${gimbal_radius}" length="${gimbal_height}"/>
+        </geometry>
+      </collision>
+    </link>
+    <joint name="gimbal_joint" type="continuous"> <!-- 修正：修改 joint 名称 -->
+      <parent link="base_link" />
+      <child link="gimbal_link" />
+      <origin xyz="0 0 ${height / 2 + gimbal_height / 2}" rpy="0 0 0" />
+      <axis xyz="0 0 1" />
+      <limit lower="-1.0" upper="1.0" effort="3.07" velocity="70" />
+    </joint>
+    <transmission name="gimbal_trans">
+      <type>transmission_interface/SimpleTransmission</type>
+      <joint name="gimbal_joint">
+        <hardwareInterface>hardware_interface/EffortJointInterface</hardwareInterface>
+      </joint>
+      <actuator name="gimbal_motor">
+        <hardwareInterface>hardware_interface/EffortJointInterface</hardwareInterface>
+        <mechanicalReduction>1</mechanicalReduction>
+      </actuator>
+    </transmission>
+    <link name="muzzle_link">
+      <inertial>
+        <origin xyz="0.0 0.0 0.0" rpy="0.0 0.0 0.0"/> <!-- 修正：质心偏移 -->
+        <mass value="0.8"/>
+        <inertia ixx="0.00036" ixy="0.0" ixz="0.0" iyy="0.01085" iyz="0.0" izz="0.0079"/>
+      </inertial>
+      <visual>
+        <origin xyz="${muzzle_height/10} 0.0 0.0" rpy="0 ${pi/2} 0"/> <!-- 修正：让枪管从关节处延伸 -->
+        <geometry>
+          <cylinder radius="${muzzle_radius}" length="${muzzle_height}"/>
+        </geometry>
+        <material name="white"/>
+      </visual>
+      <collision>
+        <origin xyz="${muzzle_height/2} 0.0 0.0" rpy="0 ${pi/2} 0"/>
+        <geometry>
+          <cylinder radius="${muzzle_radius}" length="${muzzle_height}"/>
+        </geometry>
+      </collision>
+    </link>
+    <joint name="muzzle_joint" type="revolute">
+      <parent link="gimbal_link" />
+      <child link="muzzle_link" />
+      <!-- 修正：Z 轴只需考虑相对于云台中心的高度，通常为 0 或云台顶部 -->
+      <origin xyz="0.0 0 0.15" rpy="0 0 0" />
+      <axis xyz="0 1 0" />
+      <limit lower="-0.5" upper="0.24" effort="3" velocity="70" />
+    </joint>
+    <transmission name="muzzle_trans">
+      <type>transmission_interface/SimpleTransmission</type>
+      <joint name="muzzle_joint">
+        <hardwareInterface>hardware_interface/EffortJointInterface</hardwareInterface>
+      </joint>
+      <actuator name="muzzle_motor">
+        <hardwareInterface>hardware_interface/EffortJointInterface</hardwareInterface>
+        <mechanicalReduction>1</mechanicalReduction>
+      </actuator>
+    </transmission>
+    <gazebo reference="gimbal_imu_link">
+      <gravity>true</gravity>
+      <sensor name="muzzle_imu_sensor" type="imu">
+        <always_on>true</always_on>
+        <update_rate>1000</update_rate>
+        <visualize>true</visualize>
+        <imu/>
+        <plugin filename="libgazebo_ros_imu_sensor.so" name="muzzle_imu_plugin">
+          <topicName>gimbal_imu</topicName>
+          <bodyName>gimbal_imu_link</bodyName>
+          <updateRateHZ>100.0</updateRateHZ>
+          <gaussianNoise>0.0</gaussianNoise>
+          <xyzOffset>0 0 0</xyzOffset>
+          <rpyOffset>0 0 0</rpyOffset>
+          <frameName>muzzle_link</frameName>
+          <initialOrientationAsReference>false</initialOrientationAsReference>
+        </plugin>
+      </sensor>
+    </gazebo>
     <gazebo reference="imu_link">
       <gravity>true</gravity>

Commit message: Change urdf to decline the range from center of mass and wheel axis

File: src/balance_description/urdf/balance.urdf.xacro (robot description, xacro)
@@ -106,5 +106,5 @@
       </link>
       <joint name="${prefix}_wheel_joint" type="continuous">
-        <origin xyz="0.0 ${reflect*(width/2+wheel_length/2)} ${-height*5}" rpy="${-pi/2} 0.0 0.0"/>
+        <origin xyz="0.0 ${reflect*(width/2+wheel_length/2)} ${-height*3}" rpy="${-pi/2} 0.0 0.0"/>
         <parent link="base_link"/>
         <child link="${prefix}_wheel"/>
