Commit message: Add an avalible urdf

File: src/balance_description/urdf/balance.urdf.xacro (robot description, xacro)
@@ -24,15 +24,16 @@
     <xacro:property name="thigh_length" value="0.4"/>
     <xacro:property name="shank_length" value="0.5"/>
-    <xacro:property name="leg_mass" value="0.1"/>
+    <xacro:property name="leg_mass" value="0.5"/>
     <!-- =================================================================================== -->
     <!-- Macros -->
     <!-- =================================================================================== -->
     <!-- Inertia Macros -->
-    <xacro:macro name="box_inertial" params="m w h d">
+    <xacro:macro name="box_inertial" params="m x y z ox:=0.0 oy:=0.0 oz:=0.0">
       <inertial>
+        <origin xyz="${ox} ${oy} ${oz}" rpy="0 0 0"/>
         <mass value="${m}"/>
-        <inertia ixx="${m/12 * (h*h + d*d)}" ixy="0.0" ixz="0.0"
-                 iyy="${m/12 * (w*w + d*d)}" iyz="0.0"
-                 izz="${m/12 * (w*w + h*h)}"/>
+        <inertia ixx="${m/12 * (y*y + z*z)}" ixy="0.0" ixz="0.0"
+                 iyy="${m/12 * (x*x + z*z)}" iyz="0.0"
+                 izz="${m/12 * (x*x + y*y)}"/>
       </inertial>
     </xacro:macro>
@@ -43,4 +44,12 @@
                  iyy="${m/12 * (3*r*r + h*h)}" iyz="0.0"
                  izz="${m/2 * r*r}"/>
+      </inertial>
+    </xacro:macro>
+    <xacro:macro name="cylinder_inertial_y" params="m r h">
+      <inertial>
+        <mass value="${m}"/>
+        <inertia ixx="${m/12 * (3*r*r + h*h)}" ixy="0.0" ixz="0.0"
+                 iyy="${m/2 * r*r}" iyz="0.0"
+                 izz="${m/12 * (3*r*r + h*h)}"/>
       </inertial>
     </xacro:macro>
@@ -88,5 +97,5 @@
         </collision>
         <inertial>
-            <origin xyz="-0.015 0.0 0.0" rpy="0.0 0.0 0.0"/>
+            <origin xyz="0.0 0.0 0.0" rpy="0.0 0.0 0.0"/>
             <mass value="${mass}"/>
             <inertia ixx="0.04229" ixy="0.0" ixz="0.0" iyy="0.04229" iyz="0.0" izz="0.08333"/>
@@ -98,5 +107,5 @@
             <geometry><box size="0.01 0.01 0.01"/></geometry>
         </visual>
-        <xacro:box_inertial m="0.001" w="0.01" h="0.01" d="0.01"/>
+        <xacro:box_inertial m="0.001" x="0.01" y="0.01" z="0.01"/>
     </link>
     <joint name="imu_joint" type="fixed">
@@ -145,5 +154,5 @@
         <inertial>
             <mass value="0.8"/>
-            <origin xyz="0 0 0"/>
+            <origin xyz="${muzzle_height/10} 0.0 0.0"/>
             <inertia ixx="0.00036" ixy="0.0" ixz="0.0" iyy="0.01085" iyz="0.0" izz="0.0079"/>
         </inertial>
@@ -160,5 +169,5 @@
         <geometry><box size="0.01 0.01 0.01"/></geometry>
       </visual>
-      <xacro:box_inertial m="0.001" w="0.01" h="0.01" d="0.01"/>
+      <xacro:box_inertial m="0.001" x="0.01" y="0.01" z="0.01"/>
     </link>
     <joint name="gimbal_imu_joint" type="fixed">
@@ -195,8 +204,8 @@
                 </geometry>
             </collision>
-            <xacro:box_inertial m="${leg_mass}" w="${leg_width}" h="${thigh_length}" d="${leg_thickness}"/>
+            <xacro:box_inertial m="${leg_mass}" x="${leg_width}" y="${leg_thickness}" z="${thigh_length}" oz="-0.14"/>
         </link>
         <joint name="${side}_hip_joint" type="continuous">
-            <origin xyz="0.0 ${y_offset} 0" rpy="0.0 ${PI/3} 0.0"/>
+            <origin xyz="0.0 ${y_offset} 0" rpy="0.0 ${PI/2} 0.0"/>
             <parent link="base_link"/>
             <child link="${side}_thigh_link"/>
@@ -218,5 +227,5 @@
                 </geometry>
             </collision>
-            <xacro:box_inertial m="${leg_mass}" w="${leg_width}" h="${shank_length}" d="${leg_thickness}"/>
+            <xacro:box_inertial m="${leg_mass}" x="${leg_width}" y="${leg_thickness}" z="${shank_length}" oz="-0.15"/>
         </link>
         <joint name="${side}_knee_joint" type="revolute">
@@ -235,5 +244,5 @@
                 <material name="orange"/>
             </visual>
-            <xacro:box_inertial m="0.05" w="0.04" h="0.17" d="0.01"/>
+            <xacro:box_inertial m="0.05" x="0.04" y="0.01" z="0.17"/>
         </link>
         <joint name="${side}_linkage_1_joint" type="revolute">
@@ -251,8 +260,8 @@
                 <material name="orange"/>
             </visual>
-            <xacro:box_inertial m="0.05" w="0.04" h="0.085" d="0.01"/>
+            <xacro:box_inertial m="0.05" x="0.04" y="0.01" z="0.085" oz="0.0425"/>
         </link>
         <joint name="${side}_linkage_2_joint" type="continuous">
-            <origin xyz="0 ${y_offset} 0" rpy="0 ${5*PI/6} 0"/>
+            <origin xyz="0 ${y_offset} 0" rpy="0 ${PI} 0"/>
             <parent link="base_link"/>
             <child link="${side}_linkage_2"/>
@@ -267,9 +276,9 @@
                 <material name="white"/>
             </visual>
-            <xacro:box_inertial m="0.02" w="0.02" h="0.17" d="0.01"/>
+            <xacro:box_inertial m="0.02" x="0.02" y="0.01" z="0.17" oz="0.07"/>
         </link>
         <joint name="${side}_cross_conn_1_joint" type="revolute">
-            <origin xyz="0 0 0.07" rpy="0.0 ${PI/2} 0.0"/>
-            <parent link="${side}_linkage_2"/>
+            <origin xyz="0 0 0.07" rpy="0.0 ${-PI/2} 0.0"/>
+            <parent link="${side}_linkage_1"/>
             <child link="${side}_cross_conn_1"/>
             <axis xyz="0.0 1 0.0"/>
@@ -284,5 +293,5 @@
                 <material name="white"/>
             </visual>
-             <xacro:box_inertial m="0.02" w="0.02" h="0.17" d="0.01"/>
+             <xacro:box_inertial m="0.02" x="0.02" y="0.01" z="0.17" oz="0.07"/>
         </link>
         <joint name="${side}_cross_conn_2_joint" type="revolute">
@@ -308,5 +317,5 @@
                 </geometry>
             </collision>
-            <xacro:cylinder_inertial m="${wheel_mass}" r="${wheel_radius}" h="${wheel_length}"/>
+            <xacro:cylinder_inertial_y m="${wheel_mass}" r="${wheel_radius}" h="${wheel_length}"/>
         </link>
         <joint name="${side}_wheel_joint" type="continuous">
@@ -338,10 +347,10 @@
         <joint name="${side}_cross_conn_1_loop_joint" type="revolute">
           <parent>${side}_cross_conn_1</parent>
-          <child>${side}_linkage_1</child>
+          <child>${side}_linkage_2</child>
           <axis>
             <xyz>0 1 0</xyz>
           </axis>
           <limit lower="-3.14" upper="3.14" effort="10" velocity="100"/>
-          <pose>0 0 -0.07 0 0 0</pose>
+          <pose>0 0 0.07 0 0 0</pose>
         </joint>
       </gazebo>

Commit message: Avalible ver of urdf

File: src/balance_description/urdf/balance.urdf.xacro (robot description, xacro)
@@ -203,4 +203,14 @@
             <axis xyz="0.0 1 0.0"/>
         </joint>
+        <transmission name="${side}_hip_trans">
+            <type>transmission_interface/SimpleTransmission</type>
+            <joint name="${side}_hip_joint">
+                <hardwareInterface>hardware_interface/EffortJointInterface</hardwareInterface>
+            </joint>
+            <actuator name="${side}_hip_motor">
+                <hardwareInterface>hardware_interface/EffortJointInterface</hardwareInterface>
+                <mechanicalReduction>1</mechanicalReduction>
+            </actuator>
+        </transmission>
         <!-- 2. Shank (Second Leg) -->
         <link name="${side}_shank_link">
@@ -259,4 +269,14 @@
             <axis xyz="0.0 1 0.0"/>
         </joint>
+        <transmission name="${side}_linkage_2_trans">
+            <type>transmission_interface/SimpleTransmission</type>
+            <joint name="${side}_linkage_2_joint">
+                <hardwareInterface>hardware_interface/EffortJointInterface</hardwareInterface>
+            </joint>
+            <actuator name="${side}_linkage_2_motor">
+                <hardwareInterface>hardware_interface/EffortJointInterface</hardwareInterface>
+                <mechanicalReduction>1</mechanicalReduction>
+            </actuator>
+        </transmission>
         <!-- Cross Connection 1: Connects to Linkage 2 -->
         <!-- Originally 'first_connect_complex' parent 'second_complex' (linkage_2) -->
@@ -343,5 +363,5 @@
           </axis>
           <limit lower="-3.14" upper="3.14" effort="10" velocity="100"/>
-          <pose>0 0 -0.07 0 0 0</pose>
+          <pose>0 0 0.07 0 0 0</pose>
         </joint>
       </gazebo>

Commit message: Test ver

File: src/balance_description/urdf/balance.urdf.xacro (robot description, xacro)
@@ -126,5 +126,5 @@
         <xacro:cylinder_inertial m="0.2" r="${gimbal_radius}" h="${gimbal_height}"/>
     </link>
-    <joint name="gimbal_joint" type="continuous">
+    <joint name="gimbal_joint" type="revolute">
         <parent link="base_link" />
         <child link="gimbal_link" />
@@ -371,5 +371,5 @@
             <xyz>0 1 0</xyz>
           </axis>
-          <limit lower="-3.14" upper="3.14" effort="10" velocity="100"/>
+          <limit lower="-3.14" upper="3.14" effort="3" velocity="100"/>
           <pose>0 0 0.07 0 0 0</pose>
         </joint>
@@ -382,5 +382,5 @@
             <xyz>0 1 0</xyz>
           </axis>
-          <limit lower="-3.14" upper="3.14" effort="10" velocity="100"/>
+          <limit lower="-3.14" upper="3.14" effort="3" velocity="100"/>
           <pose>0 0 0.07 0 0 0</pose>
         </joint>

Commit message: Add a support and test ik&fk

File: src/balance_description/urdf/balance.urdf.xacro (robot description, xacro)
@@ -390,4 +390,34 @@
     <xacro:leg side="left" reflect="1" />
     <xacro:leg side="right" reflect="-1" />
+    <link name="support">
+        <inertial>
+            <origin xyz="0.0 0.0 0.0" rpy="0.0 0.0 0.0"/>
+            <mass value="1000.0"/>
+            <inertia ixx="0.0" ixy="0.0" ixz="0.0" iyy="0.0" iyz="0.0" izz="0.0"/>
+        </inertial>
+        <visual name="">
+            <origin xyz="0.0 0.0 0.0" rpy="0.0 0.0 0.0"/>
+            <geometry>
+                <box size="0.5 0.3 1.0"/>
+            </geometry>
+            <material name="">
+                <color rgba="1.0 0.0 0.0 1.0"/>
+                <texture filename=""/>
+            </material>
+        </visual>
+        <collision>
+            <origin xyz="0.0 0.0 0.0" rpy="0.0 0.0 0.0"/>
+            <geometry>
+                <box size="0.5 0.3 1.0"/>
+            </geometry>
+        </collision>
+    </link>
+    <joint name="support_joint" type="fixed">
+        <origin xyz="0.0 0.0 -0.5" rpy="0.0 0.0 0.0"/>
+        <parent link="base_link"/>
+        <child link="support"/>
+        <axis xyz="0.0 0.0 0.0"/>
+        <limit lower="0.0" upper="0.0" effort="0.0" velocity="0.0"/>
+    </joint>
     <!-- =================================================================================== -->
     <!-- Gazebo Plugins -->
